File: hw/pcb/solarsat/solarsat.kicad_pcb (KiCad board)
At the start: 2 copper layers, 20 x 20 mm, 28 parts, among them J1 Conn_01x01, J10 Conn_01x01, J11 Conn_01x01, J12 Conn_01x01, J13 Conn_01x01, J2 Conn_02x03_Odd_Even, J3 Conn_01x01, J4 Conn_01x01, J5 Conn_01x01, J6 Conn_01x01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

Commit message: first routing
Parts:
- moved R6 3.64 mm to (138.3, 89.3), turned to 90 degrees
- moved R4 2.95 mm to (140.6, 89.3), turned to 90 degrees
- moved R5 2.34 mm to (139.4, 89.3), turned to 270 degrees
- moved J2 1.02 mm to (128.9, 80.6)
- moved C1 1.02 mm to (128.9, 86.5)
- moved C5 0.97 mm to (139.4, 86.7), turned to 270 degrees
- moved C6 0.46 mm to (140.6, 84.8), turned to 90 degrees
Routing:
- net GND: track 0.00 -> 31.8 mm, vias 0 -> 14
- net VBUS: track 0.00 -> 24.5 mm, vias 0 -> 3
- net Net-(C3-Pad1): track 0.00 -> 15.1 mm, vias 0 -> 2
- net Net-(J2-Pad4): track 0.00 -> 13.4 mm
- net Net-(J2-Pad3): track 0.00 -> 11.7 mm
- net Net-(J7-Pad1): track 0.00 -> 10.1 mm
- net Net-(JP1-Pad2): track 0.00 -> 9.89 mm, vias 0 -> 2
- net /LDO1: track 0.00 -> 8.87 mm
- net Net-(J2-Pad2): track 0.00 -> 8.74 mm
- net Net-(J6-Pad1): track 0.00 -> 8.72 mm
- net Net-(J8-Pad1): track 0.00 -> 7.34 mm
- net +BATT: track 0.00 -> 6.89 mm
- net /LDO2: track 0.00 -> 6.80 mm
- net Net-(L1-Pad2): track 0.00 -> 6.12 mm
- net Net-(R5-Pad2): track 0.00 -> 5.84 mm
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- added copper zone on B.Cu, net GND
Other:
- net class Default: clearance 0.2 -> 0.1524
- rule trace_clearance: 0.2 -> 0.1524
- rule trace_min: 0.2 -> 0.1524
- rule via_min_drill: 0.3 -> 0.254
- rule via_min_size: 0.4 -> 0.508

Commit message: routed
Parts:
- moved JP1 0.51 mm to (140.6, 76.7)
Routing:
- net GND: track 31.8 -> 34.6 mm
- net VBUS: track 24.5 -> 26.0 mm
Other:
- outline, holes or cut-outs redrawn
- board text added: "+BATT"
- board text added: "1"
- board text added: "2"
- board text added: "3"
- board text added: "4"
- board text added: "5"
- board text added: "6"
- board text added: "GND"
- board text added: "Jonas 2021"
- board text added: "LDO1 1.8 V"
- board text added: "LDO1 EN"
- board text added: "LDO2 3.3 V"
- board text added: "LDO2 EN"
- board text added: "VBUS"
- board text added: "~CHG"
- board text added: "~CONN"
